File: Kicad/StepperDrivers.sch (KiCad schematic (older format))
At the start: 0 parts

Commit message: Added stepper driver and componets and power management
Parts:
- added C? (x3): 100nF, symbol Device:C
- added C?: 4.7µF, symbol Device:C
- added C?: 470nF, symbol Device:C
- added C?: 100µF, symbol Device:CP
- added C?: 22nF63V, symbol Device:C
- added J?: ZAXIS, symbol Connector:Conn_01x04_Male
- added R?: 2R2, symbol Device:R
- added R? (x2): 0.5W1206, symbol Device:R
- added U? (x3): TMC2130-TA, Package_QFP:TQFP-48-1EP_7x7mm_P0.5mm_EP5x5mm, symbol Driver_Motor:TMC2130-TA
Connections:
- new net: U?.13 (GNDP), U?.48 (GNDP) (x2)
- new net: U?.31 (GNDD), U?.36 (GNDD), U?.49 (GNDD), U?.6 (GNDD) (x2)
- new net: J?.1 (Pin_1), U?.15 (OB1)
- new net: R?.2, U?.17 (BRB)
- new net: J?.2 (Pin_2), U?.19 (OB2)
- new net: C?.2, R?.2, U?.33 (5VOUT)
- new net: C?.2, R?.1, U?.34 (VCC)
- new net: C?.1, U?.35 (CPO)
- new net: C?.2, U?.37 (CPI)
- new net: C?.2, U?.38 (VCP)
- new net: J?.3 (Pin_3), U?.42 (OA2)
- new net: R?.1, U?.44 (BRA)
- new net: J?.4 (Pin_4), U?.46 (OA1)
- new net +24V: C?.1, C?.1, C?.1, U?.21 (VS), U?.39 (VSA), U?.40 (VS)
- new net +3V3: C?.1, U?.10 (VCC_IO)
- new net CS_X: U?.3 (~CS~_CFG3)
- new net CS_Y: U?.3 (~CS~_CFG3)
- new net CS_Z: U?.3 (~CS~_CFG3)
- new net GND: C?.1, C?.1, C?.2, C?.2, C?.2, R?.1, R?.2, U?.13 (GNDP), U?.2 (CLK), U?.29 (~DRV_EN~_CFG6), U?.31 (GNDD), U?.36 (GNDD), U?.48 (GNDP), U?.49 (GNDD), U?.6 (GNDD)
- new net GNDA: U?.32 (GNDA)
- new net SCK: U?.4 (SCK_CFG2), U?.4 (SCK_CFG2), U?.4 (SCK_CFG2)
- new net SDI: U?.5 (SDI_CFG1), U?.5 (SDI_CFG1), U?.5 (SDI_CFG1)
- new net SDO: U?.7 (SDO_CFG0), U?.7 (SDO_CFG0), U?.7 (SDO_CFG0)
Other:
- note added: "X-axis"
- note added: "Y-axis"
- note added: "Z-axis"
