File: Kicad/stm32.sch (KiCad schematic (older format))
At the start: 8 parts

Commit message: Added TMC2130 to board and routed
Parts:
- gave numbers to parts that had none: 8
Changed lines of the file:
@@
 EESchema Schematic File Version 4
+LIBS:Controllerboard-cache
 EELAYER 30 0
 EELAYER END
@@
 $EndDescr
 $Comp
-L Device:C C?
+L Device:C C1
 U 1 1 5E1D1E70
 P 4050 3050
-F 0 "C?" V 3798 3050 50  0000 C CNN
+F 0 "C1" V 3798 3050 50  0000 C CNN
 F 1 "12pF" V 3889 3050 50  0000 C CNN
 F 2 "" H 4088 2900 50  0001 C CNN
@@
 $EndComp
 $Comp
-L Device:C C?
+L Device:C C2
 U 1 1 5E1D2F5F
 P 4050 3450
-F 0 "C?" V 3798 3450 50  0000 C CNN
+F 0 "C2" V 3798 3450 50  0000 C CNN
 F 1 "12pF" V 3889 3450 50  0000 C CNN
 F 2 "" H 4088 3300 50  0001 C CNN
@@
 $EndComp
 $Comp
-L Device:Crystal Y?
+L Device:Crystal Y1
 U 1 1 5E1D4120
 P 4300 3250
-F 0 "Y?" V 4254 3381 50  0000 L CNN
+F 0 "Y1" V 4254 3381 50  0000 L CNN
 F 1 "8Mhz" V 4345 3381 50  0000 L CNN
 F 2 "" H 4300 3250 50  0001 C CNN
@@
 	4700 3200 5050 3200
 $Comp
-L PrivateLib:STM32F103RCTx U?
+L PrivateLib:STM32F103RCTx U1
 U 1 1 5E1DA77D
 P 5750 3500
-F 0 "U?" H 5750 2250 50  0000 C CNN
+F 0 "U1" H 5750 2250 50  0000 C CNN
 F 1 "STM32F103RCTx" H 5750 2150 50  0000 C CNN
 F 2 "Package_QFP:LQFP-64_10x10mm_P0.5mm" H 5150 1800 50  0001 R CNN
@@
 	4300 3450 4700 3450
 $Comp
-L Device:C C?
+L Device:C C4
 U 1 1 5E1DE8F8
 P 9650 2250
-F 0 "C?" H 9535 2204 50  0000 R CNN
+F 0 "C4" H 9535 2204 50  0000 R CNN
 F 1 "100nF" H 9535 2295 50  0000 R CNN
 F 2 "" H 9688 2100 50  0001 C CNN
@@
 $EndComp
 $Comp
-L Device:C C?
+L Device:C C5
 U 1 1 5E1DF543
 P 10100 2250
-F 0 "C?" H 9985 2204 50  0000 R CNN
+F 0 "C5" H 9985 2204 50  0000 R CNN
 F 1 "100nF" H 9985 2295 50  0000 R CNN
 F 2 "" H 10138 2100 50  0001 C CNN
@@
 $EndComp
 $Comp
-L Device:C C?
+L Device:C C6
 U 1 1 5E1DF8BC
 P 10550 2250
-F 0 "C?" H 10435 2204 50  0000 R CNN
+F 0 "C6" H 10435 2204 50  0000 R CNN
 F 1 "100nF" H 10435 2295 50  0000 R CNN
 F 2 "" H 10588 2100 50  0001 C CNN
@@
 $EndComp
 $Comp
-L Device:C C?
+L Device:C C3
 U 1 1 5E1DFC3F
 P 9200 2250
-F 0 "C?" H 9085 2204 50  0000 R CNN
+F 0 "C3" H 9085 2204 50  0000 R CNN
 F 1 "100nF" H 9085 2295 50  0000 R CNN
 F 2 "" H 9238 2100 50  0001 C CNN
