File: Kicad/_autosave-Controllerboard.kicad_pcb (KiCad board)
At the start: 2 copper layers, 100 x 80 mm, 53 parts, among them J1 Conn_01x02_Male, J3 ZAXIS, J4 XAXIS, J5 YAXIS, Q1 Q_PMOS_DSG, Q2 Q_NMOS_GDS, U1 STM32F103RCTx, U2 LM5155, U3 AMS1117-3.3, U4 TMC2130-TA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

Commit message: Completed the TMC2130 layout and Boost converter layout
Parts:
- added D3: D, PrivateLib:DPAK, F.Cu at (140.0, 87.0)
- added M1: Motor_DC, PrivateLib:XT30PW-M, F.Cu at (141.0, 81.2)
- added Q3: Q_NMOS_DSG, Package_TO_SOT_SMD:TO-252-2, F.Cu at (143.8, 97.0)
- added R12: 10k, Resistor_SMD:R_0603_1608Metric, F.Cu at (157.0, 128.8)
- added R13: 0.01R, Resistor_SMD:R_1206_3216Metric, F.Cu at (157.2, 124.8)
Routing:
- net Net-(D2-Pad2): track 0.00 -> 18.4 mm
- net +VDC: track 48.5 -> 60.5 mm
- net Net-(F1-Pad2): track 0.70 -> 5.70 mm
- net Net-(F1-Pad1): track 0.00 -> 4.11 mm
- net GND: vias 49 -> 52
